Commit message: Define gripper macro for the pg70
By this change the macro prbt_gripper has to be instantiated, instead of only including the xacro file.

File: prbt_pg70_support/urdf/pg70.urdf.xacro (robot description, xacro)
@@ -12,12 +12,12 @@
 limitations under the License.
 -->
-<gripper name="pg70" xmlns:xacro="http://www.ros.org/wiki/xacro">
-  <!-- Load pg70 gripper macro -->
-  <xacro:include filename="$(find schunk_description)/urdf/pg70/pg70.urdf.xacro" />
-  <!-- name of the gripper -->
-  <xacro:arg name="gripper_name" default="$(arg robot_prefix)gripper"/>
-  <!-- instantiate the gripper -->
-  <xacro:schunk_pg70 parent="$(arg robot_prefix)flange" name="$(arg gripper_name)" has_podest="false">
-    <origin xyz="0 0 0.0171" rpy="0 0 ${-pi*3/4.}" />
-  </xacro:schunk_pg70>
+<gripper xmlns:xacro="http://www.ros.org/wiki/xacro">
+  <xacro:macro name="prbt_gripper" params="gripper_name:=^ parent">
+    <!-- Load pg70 gripper macro -->
+    <xacro:include filename="$(find schunk_description)/urdf/pg70/pg70.urdf.xacro" />
+    <!-- instantiate the gripper -->
+    <xacro:schunk_pg70 parent="${parent}" name="${gripper_name}" has_podest="false">
+      <origin xyz="0 0 0.0171" rpy="0 0 ${-pi*3/4.}" />
+    </xacro:schunk_pg70>
+  </xacro:macro>
 </gripper>
